Commit message: added config file to set the urdf path

File: urdf/youbot_model.urdf (robot description, URDF)
Before this commit: robot youbot, 51 links, 50 joints
Links:
- link arm_link_5: mass 0.387 -> 0.687

Commit message: ROS2 port

File: urdf/youbot_model.urdf (robot description, URDF)
Before this commit: robot youbot, 51 links, 50 joints
Links:
- link arm_link_5: mass 0.687 -> 0.887
